File: hardware/emmc-type-c-version/sdcdmuxemmc-ifrc.kicad_sch (KiCad schematic)
At the start: 11 parts, among them Q201 2N7002K, U201 TSSP4038

Commit message: Corrected part number in the BOM
Parts:
- C201: digikey 311-3494-1-ND -> 311-1355-1-ND; storeURL https://www.digikey.com/en/products/detail/yageo/CC0603MRX5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 -> https://www.digikey.com/en/products/detail/yageo/CC0805ZKY5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
- C202: footprint Capacitor_SMD:C_0805_2012Metric_Pad1.18x1.45mm_HandSolder -> Capacitor_SMD:C_0603_1608Metric_Pad1.08x0.95mm_HandSolder; digikey 311-3494-1-ND -> 311-1815-1-ND; storeURL https://www.digikey.com/en/products/detail/yageo/CC0603MRX5R8BB106/7164378 -> https://www.digikey.com/en/products/detail/yageo/CC0603MRX5R5BB226/519522
- R201, R205: footprint tbctl:R_0805_2012Metric_Pad1.20x1.40mm_HandSolder -> Resistor_SMD:R_0805_2012Metric_Pad1.20x1.40mm_HandSolder; digikey 13-RC0603JR-1010KLCT-ND -> 311-10KARCT-ND; storeURL https://www.digikey.com/en/products/detail/yageo/RC0603JR-1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 -> https://www.digikey.com/en/products/detail/yageo/RC0805JR-0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
- R202: footprint tbctl:R_0805_2012Metric_Pad1.20x1.40mm_HandSolder -> Resistor_SMD:R_0805_2012Metric_Pad1.20x1.40mm_HandSolder; digikey 13-RC0603JR-101KLCT-ND -> 311-1.0KARCT-ND; storeURL https://www.digikey.com/en/products/detail/yageo/RC0603JR-1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 -> https://www.digikey.com/en/products/detail/yageo/RC0805JR-0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
- R204: footprint tbctl:R_0805_2012Metric_Pad1.20x1.40mm_HandSolder -> Resistor_SMD:R_0805_2012Metric_Pad1.20x1.40mm_HandSolder; digikey 13-RC0603JR-1010KLCT-ND -> 311-100ARCT-ND; storeURL https://www.digikey.com/en/products/detail/yageo/RC0603JR-1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 -> https://www.digikey.com/en/products/detail/yageo/RC0805JR-0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
