File: hardware/emmc-type-c-version/sdcdmuxemmc-mux.kicad_sch (KiCad schematic)
At the start: 12 parts, among them U601 TMUX1574PWR, U602 TMUX1574PWR, U603 TMUX1574PWR, U604 EM32VSUKN

Commit message: Corrected part number in the BOM
Parts:
- C604, C605: digikey 13-CC0603KPX7R7BB105CT-ND -> 311-3440-1-ND; storeURL https://www.digikey.com/en/products/detail/yageo/CC0603KPX7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 -> https://www.digikey.com/en/products/detail/yageo/CC0805MRY5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
- R601, R602: footprint tbctl:R_0805_2012Metric_Pad1.20x1.40mm_HandSolder -> Resistor_SMD:R_0805_2012Metric_Pad1.20x1.40mm_HandSolder; digikey 13-RC0603JR-1010KLCT-ND -> 311-10KARCT-ND; storeURL https://www.digikey.com/en/products/detail/yageo/RC0603JR-1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 -> https://www.digikey.com/en/products/detail/yageo/RC0805JR-0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
