File: hardware/emmc-type-c-version/sdcdmuxemmc-usbif.kicad_sch (KiCad schematic)
At the start: 21 parts, among them U401 AT24MAC402-STUM, U402 USB2640-HZH-02, Y401 24MHz

Commit message: Corrected part number in the BOM
Parts:
- C401, C402, C409, C410: footprint tbctl:C_0805_2012Metric_Pad1.18x1.45mm_HandSolder -> Capacitor_SMD:C_0805_2012Metric_Pad1.18x1.45mm_HandSolder; digikey 13-CC0603KPX7R7BB105CT-ND -> 311-3440-1-ND; storeURL https://www.digikey.com/en/products/detail/yageo/CC0603KPX7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 -> https://www.digikey.com/en/products/detail/yageo/CC0805MRY5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
- C411, C412: footprint tbctl:C_0805_2012Metric_Pad1.18x1.45mm_HandSolder -> Capacitor_SMD:C_0805_2012Metric_Pad1.18x1.45mm_HandSolder; digikey 311-1455-1-ND -> 490-14466-1-ND; storeURL https://www.digikey.com/en/products/detail/yageo/CC0603KRX5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 -> https://www.digikey.com/en/products/detail/murata-electroni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
- R401: footprint tbctl:R_0805_2012Metric_Pad1.20x1.40mm_HandSolder -> Resistor_SMD:R_0805_2012Metric_Pad1.20x1.40mm_HandSolder; digikey 311-1.0MGRCT-ND -> 311-1.0MARCT-ND; storeURL https://www.digikey.com/en/products/detail/yageo/RC0603JR-0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 -> https://www.digikey.com/en/products/detail/yageo/RC0805JR-0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
- R402: footprint tbctl:R_0805_2012Metric_Pad1.20x1.40mm_HandSolder -> Resistor_SMD:R_0805_2012Metric_Pad1.20x1.40mm_HandSolder; digikey 311-12.0KHRCT-ND -> 311-12.0KCRCT-ND; storeURL https://www.digikey.com/en/products/detail/yageo/RC0603FR-0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 -> https://www.digikey.com/en/products/detail/yageo/RC0805FR-0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
- R403, R404: footprint tbctl:R_0805_2012Metric_Pad1.20x1.40mm_HandSolder -> Resistor_SMD:R_0805_2012Metric_Pad1.20x1.40mm_HandSolder; digikey 13-RC0603JR-1010KLCT-ND -> 311-10KARCT-ND; storeURL https://www.digikey.com/en/products/detail/yageo/RC0603JR-1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 -> https://www.digikey.com/en/products/detail/yageo/RC0805JR-0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
- R405: footprint tbctl:R_0805_2012Metric_Pad1.20x1.40mm_HandSolder -> Resistor_SMD:R_0805_2012Metric_Pad1.20x1.40mm_HandSolder; digikey 311-330GRCT-ND -> 311-330ARCT-ND; storeURL https://www.digikey.com/en/products/detail/yageo/RC0603JR-0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 -> https://www.digikey.com/en/products/detail/yageo/RC0805JR-0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
